File: hardware/SFP Doctor.kicad_pcb (KiCad board)
At the start: 2 copper layers, 55 x 87.8 mm, 19 parts, among them J1 1888247-1, P1 CONN_01X26, P2 CONN_01X26, U1 TSR_1-2433, U2 PCA9306

Commit message: wip: revision 1.2 of PCB
Parts:
- removed R6, R8: 0R (NU), Resistor_SMD:R_1206_3216Metric_Pad1.42x1.75mm_HandSolder
- removed R7, R9: 0R, Resistor_SMD:R_1206_3216Metric_Pad1.42x1.75mm_HandSolder
- added D1: APA102, LED_SMD:LED_RGB_5050-6, F.Cu at (59.5, 117.9)
- added D2: APA102, LED_SMD:LED_RGB_5050-6, F.Cu at (66.7, 117.9)
- added D3: APA102, LED_SMD:LED_RGB_5050-6, F.Cu at (73.9, 117.9)
- C1, C2: value C -> 100nF
- J1: value 1888247-1 -> 2227023-1; footprint 1888247-1:TE_1888247-1 -> 2227023-1:TE_2227023-1
- moved G*** 24.1 mm to (90.0, 110.8)
- moved C1 2.30 mm to (80.7, 54.2)
- moved R1 0.50 mm to (87.5, 52.5)
- turned J1 to 90 degrees
Connections:
- P1 pad 11: SDA_0_5V -> Net-(P1-Pad11)
- P1 pad 12: SCL_0_5V -> Net-(P1-Pad12)
- P1 pad 15: SDA_1_5V -> SDA_5V
- P1 pad 16: SCL_1_5V -> SCL_5V
- P1 pad 22: Net-(P1-Pad22) -> LED_CLOCK
- P1 pad 23: Net-(P1-Pad23) -> LED_DATA
Routing:
- net GND: track 147.4 -> 9.95 mm, vias 0 -> 18
- net +5V: track 37.5 -> 136.1 mm
- net LED_CLOCK: track 0.00 -> 37.3 mm
- net LED_DATA: track 0.00 -> 28.4 mm
- net +3V3: track 42.6 -> 54.1 mm, vias 0 -> 2
- net Net-(D1-Pad6): track 0.00 -> 11.4 mm
- net Net-(D1-Pad5): track 0.00 -> 11.3 mm
- net Net-(D2-Pad5): track 0.00 -> 10.9 mm
- net Net-(D2-Pad6): track 0.00 -> 10.2 mm
- net SCL_1_5V: track 9.23 -> 0.00 mm
- net SCL_0_5V: track 9.21 -> 0.00 mm
- net SDA_0_5V: track 8.94 -> 0.00 mm
- net SDA_1_5V: track 8.80 -> 0.00 mm
- net SDA_3V3: track 30.4 -> 33.6 mm
- net SCL_5V: track 88.5 -> 85.8 mm, vias 4 -> 3
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- added copper zone on B.Cu, net GND
- added copper zone on F.Cu, net GND
Other:
- board text added: "Operation"
- board text added: "Rev. 1.2"
- board text added: "Search"
- board text added: "Status"
- board text removed: "Rev. 1.0"

Commit message: wip: revision 1.3 of PCB
Moved SFP cage
Parts:
- moved D1 56.1 mm to (83.5, 67.2)
- moved D2 56.1 mm to (90.7, 67.2)
- moved D3 56.1 mm to (97.9, 67.2)
- moved J1 26.4 mm to (91.3, 88.3)
- moved G*** 24.3 mm to (65.8, 110.4)
Connections:
- P1 pad 22: LED_CLOCK -> Net-(P1-Pad22)
- P1 pad 23: LED_DATA -> Net-(P1-Pad23)
- P2 pad 11: Net-(P2-Pad11) -> LED_DATA
- P2 pad 12: Net-(P2-Pad12) -> LED_CLOCK
Routing:
- net +5V: track 136.1 -> 82.9 mm, vias 1 -> 3
- net LED_CLOCK: track 37.3 -> 7.87 mm
- net SCL_3V3: track 26.3 -> 52.5 mm
- net SDA_3V3: track 33.6 -> 59.3 mm
- net +3V3: track 54.1 -> 78.2 mm
- net LED_DATA: track 28.4 -> 5.38 mm
- net SCL_5V: track 85.8 -> 84.5 mm
- net Net-(P2-Pad13): track 0.00 -> 1.20 mm
- net SDA_5V: track 85.3 -> 86.1 mm
Other:
- board text added: "Rev. 1.3"
- board text removed: "Rev. 1.2"
